File: flipcab.kicad_pcb (KiCad board)
At the start: 2 copper layers, 50 x 23 mm, 37 parts, among them J1 LED, J2 USB_JTAG, J3 MOTOR_OUT, SW1 OPEN_DET, SW2 CLOSE_DET, SW3 BOOT, U1 ESP32-C6-MINI-1, U2 AL8860MP, U3 CH221K, U4 DRV8870DDA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

Commit message: rev1: sync change
Parts:
- removed the C7 at (140.1, 79.8)
- removed D1: SS24FL, Diode_SMD:D_SOD-123F
- removed the J3 at (132.4, 104.0)
- removed R13, R14: 5.11k, Resistor_SMD:R_0402_1005Metric
- removed the R4 at (114.9, 119.3)
- removed the R5 at (117.8, 113.3)
- removed Y1: 32.768k, Crystal:Crystal_SMD_3215-2Pin_3.2x1.5mm
- added C10: 100nF, Capacitor_SMD:C_0402_1005Metric, F.Cu at (92.5, 100.4)
- added J2: UART_PROG, Connector_PinHeader_1.27mm:PinHeader_1x06_P1.27mm_Vertical, F.Cu at (91.1, 83.9)
- added J4: MOTOR_OUT, Connector_PinHeader_2.54mm:PinHeader_1x02_P2.54mm_Vertical, F.Cu at (96.7, 101.0)
- added Q1: AO3400A, Package_TO_SOT_SMD:SOT-23, F.Cu at (108.2, 108.8)
- added R11: 5.11k, Resistor_SMD:R_0402_1005Metric, F.Cu at (107.2, 112.0)
- C4: footprint Capacitor_SMD:C_0402_1005Metric -> Capacitor_SMD:C_0603_1608Metric
- C6: value 20pF -> 100nF
- C7: renamed from C8; value 1uF -> 22uF
- C8: renamed from C10; value 100nF -> 1uF; footprint Capacitor_SMD:C_0402_1005Metric -> Capacitor_SMD:C_0603_1608Metric
- J1: value LED -> LED_OUT
- L1: value 47uH -> 3.9uH; footprint Inductor_SMD:L_APV_ANR6045 -> Inductor_SMD:L_Changjiang_FNR3015S
- R10: renamed from R11; value 20k -> 100mR/0.5w; footprint Resistor_SMD:R_0402_1005Metric -> Resistor_SMD:R_1206_3216Metric
- R7: renamed from R9; value 0.15R/0.5w -> 1k; footprint Resistor_SMD:R_0805_2012Metric -> Resistor_SMD:R_0402_1005Metric
- R8: renamed from R10; value 1k -> 47k
- R9: renamed from R12; value 100mR/0.5w -> 5.11k; footprint Resistor_SMD:R_1206_3216Metric -> Resistor_SMD:R_0402_1005Metric
- U2: value AL8860MP -> AP63203WU; footprint Package_SO:MSOP-8-1EP_3x3mm_P0.65mm_EP1.5x1.8mm -> Package_TO_SOT_SMD:TSOT-23-6
- moved C6 87.6 mm to (54.6, 96.8)
- moved C7 83.6 mm to (57.3, 96.5), turned to 180 degrees
- moved U2 79.1 mm to (52.3, 99.1)
- moved C9 76.6 mm to (62.5, 98.3), turned to -90 degrees
- moved C8 73.4 mm to (68.0, 95.6), turned to -90 degrees
- moved R7 71.2 mm to (69.7, 92.5), turned to -90 degrees
- moved C3 68.7 mm to (72.4, 81.0), turned to 180 degrees
- moved C2 67.9 mm to (74.3, 88.9), turned to -90 degrees
- moved C1 67.5 mm to (73.8, 82.7), turned to 180 degrees
- moved C5 54.8 mm to (87.8, 92.2)
- moved R3 53.7 mm to (73.0, 83.8)
- moved R2 53.1 mm to (68.2, 90.1)
- moved R8 53.0 mm to (71.8, 93.2)
- moved R1 48.4 mm to (74.3, 86.9), turned to -90 degrees
- moved R6 42.3 mm to (83.8, 92.2)
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- renumbered J2 to J3, R6 to R4, R8 to R5, R7 to R6
Connections:
- C4 pad 1: +9V -> +12V
- C6 pad 1: GND -> Net-(U2-BST)
- C6 pad 2: IO0 -> Net-(U2-SW)
- C7 pad 1: Net-(U3-VDD) -> +3V3
- C8 pad 1: GND -> Net-(U3-VDD)
- C8 pad 2: +9V -> GND
- C9 pad 1: +9V -> +12V
- J1 pad 2: Net-(J1-Pin_2) -> +12V
- J3 pad A4: +9V -> +12V
- J3 pad A9: +9V -> +12V
- J3 pad B4: +9V -> +12V
- J3 pad B9: +9V -> +12V
- L1 pad 1: Net-(J1-Pin_1) -> Net-(U2-SW)
- L1 pad 2: Net-(D1-A) -> +3V3
- R10 pad 1: Net-(U3-VDD) -> Net-(U4-ISEN)
- R10 pad 2: Net-(U3-CFG) -> GND
- R2 pad 1: Net-(SW1-C) -> Net-(SW1-A)
- R2 pad 2: +3V3 -> OPEN_SW
- R3 pad 1: GND -> Net-(SW2-A)
- R3 pad 2: Net-(SW1-B) -> CLOSE_SW
- R7 pad 1: +9V -> +12V
- R7 pad 2: Net-(J1-Pin_2) -> Net-(U3-VDD)
- R8 pad 1: +9V -> Net-(U3-VDD)
- R8 pad 2: Net-(U3-VDD) -> Net-(U3-CFG)
- R9 pad 1: Net-(U4-ISEN) -> CC2
- SW1 pad 1: OPEN_SW -> Net-(SW1-A)
- SW1 pad 2: Net-(SW1-B) -> GND
- SW1 pad 3: Net-(SW1-C) -> +3V3
- SW2 pad 1: CLOSE_SW -> Net-(SW2-A)
- SW2 pad 2: Net-(SW2-B) -> GND
- SW2 pad 3: Net-(SW2-C) -> +3V3
- U1 pad 10: IO5 -> unconnected-(U1-IO5-Pad10)
- U1 pad 12: IO0 -> unconnected-(U1-IO0-Pad12)
- U1 pad 13: IO1 -> unconnected-(U1-IO1-Pad13)
- U1 pad 15: LPI2C_SDA -> unconnected-(U1-IO6-Pad15)
- U1 pad 16: LPI2C_SCL -> unconnected-(U1-IO7-Pad16)
- U1 pad 19: STATE_LED -> LED_CTRL
- U1 pad 9: IO4 -> unconnected-(U1-IO4-Pad9)
- U2 pad 1: Net-(J1-Pin_2) -> +3V3
- U2 pad 2: GND -> +12V
- U2 pad 3: GND -> +12V
- U2 pad 4: LED_CTRL -> GND
- U2 pad 5: Net-(D1-A) -> Net-(U2-SW)
- U2 pad 6: Net-(D1-A) -> Net-(U2-BST)
- U4 pad 5: +9V -> +12V
Routing:
- net GND: track 0.00 -> 11.2 mm
- net CC2: track 0.00 -> 10.6 mm
- net Net-(J4-Pin_2): track 0.00 -> 8.61 mm
- net +3V3: track 0.00 -> 7.03 mm, vias 0 -> 2
- net IO9/BOOT: track 0.00 -> 6.30 mm
- net Net-(J4-Pin_1): track 0.00 -> 6.02 mm
- net Net-(U3-VDD): track 0.00 -> 5.04 mm
- net Net-(U2-SW): track 0.00 -> 4.43 mm
- net UART_RXD: track 0.00 -> 3.59 mm
- net UART_TXD: track 0.00 -> 3.39 mm
- net Net-(U4-ISEN): track 0.00 -> 3.00 mm
- net MOTOR_IN1: track 0.00 -> 2.85 mm, vias 0 -> 2
- net EN: track 0.00 -> 2.82 mm
- net MOTOR_IN2: track 0.00 -> 2.80 mm, vias 0 -> 2
- net IO8: track 0.00 -> 2.09 mm
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Other:
- copper layers 2 -> 4
