File: flipcab.kicad_sch (KiCad schematic)
At the start: 0 parts

Commit message: rev1: finish schmetic
Parts:
- added C1, C2: 1uF, Capacitor_SMD:C_0402_1005Metric, symbol Device:C
- added C10, C5: 100nF, Capacitor_SMD:C_0402_1005Metric, symbol Device:C
- added C3: 22uF, Capacitor_SMD:C_0603_1608Metric, symbol Device:C
- added C4: 10uF, Capacitor_SMD:C_0402_1005Metric, symbol Device:C
- added C6, C7: 20pF, Capacitor_SMD:C_0402_1005Metric, symbol Device:C
- added C8: 1uF, Capacitor_SMD:C_0603_1608Metric, symbol Device:C
- added C9: 47uF, Capacitor_Tantalum_SMD:CP_EIA-7343-31_Kemet-D, symbol Device:C_Polarized
- added D1: SS24FL, Diode_SMD:D_SOD-123F, symbol Device:D
- added J1: LED, Connector_PinHeader_2.54mm:PinHeader_1x02_P2.54mm_Vertical, symbol Connector:Conn_01x02_Pin
- added J2: USB_JTAG, Connector_USB:USB_C_Receptacle_HRO_TYPE-C-31-M-12, symbol Connector:USB_C_Receptacle_USB2.0
- added J3: MOTOR_OUT, Connector_PinHeader_2.54mm:PinHeader_1x02_P2.54mm_Vertical, symbol Connector:Conn_01x02_Pin
- added L1: 47uH, Inductor_SMD:L_APV_ANR6045, symbol Device:L
- added R1, R7: 10k, Resistor_SMD:R_0402_1005Metric, symbol Device:R
- added R10: 1k, Resistor_SMD:R_0402_1005Metric, symbol Device:R
- added R11: 20k, Resistor_SMD:R_0402_1005Metric, symbol Device:R
- added R12: 100mR/0.5w, Resistor_SMD:R_1206_3216Metric, symbol Device:R
- added R13, R14: 5.11k, Resistor_SMD:R_0402_1005Metric, symbol Device:R_Small
- added R2, R3, R4, R5, R6, R8: 22k, Resistor_SMD:R_0402_1005Metric, symbol Device:R
- added R9: 0.15R/0.5w, Resistor_SMD:R_0805_2012Metric, symbol Device:R
- added SW1: OPEN_DET, Button_Switch_THT:SW_XKB_DM1-16UP-1, symbol Switch:SW_SPDT_XKB_DMx-xxxx-1
- added SW2: CLOSE_DET, Button_Switch_THT:SW_XKB_DM1-16UP-1, symbol Switch:SW_SPDT_XKB_DMx-xxxx-1
- added SW3: BOOT, Button_Switch_SMD:SW_Push_1P1T_XKB_TS-1187A, symbol Switch:SW_Push
- added U1: ESP32-C6-MINI-1, RF_Module:ESP32-C6-MINI-1, symbol RF_Module:ESP32-C6-MINI-1
- added U2: AL8860MP, Package_SO:MSOP-8-1EP_3x3mm_P0.65mm_EP1.5x1.8mm, symbol Driver_LED:AL8860MP
- added U3: CH221K, Package_TO_SOT_SMD:SOT-23-6, symbol JackcoLib:CH221K
- added U4: DRV8870DDA, Package_SO:Texas_HTSOP-8-1EP_3.9x4.9mm_P1.27mm_EP2.95x4.9mm_Mask2.4x3.1mm_ThermalVias, symbol Driver_Motor:DRV8870DDA
- added Y1: 32.768k, Crystal:Crystal_SMD_3215-2Pin_3.2x1.5mm, symbol Device:Crystal
Connections:
- new net: J3.1 (Pin_1), U4.6 (OUT1)
- new net: R12.1, U4.7 (ISEN)
- new net: J3.2 (Pin_2), U4.8 (OUT2)
- new net: C8.1, R10.2, R11.1, U3.1 (VDD)
- new net: J1.1 (Pin_1), L1.1
- new net: D1.2 (A), L1.2, U2.5 (SW), U2.6 (SW)
- new net: J1.2 (Pin_2), R9.2, U2.1 (SET)
- new net: R3.2, SW1.2 (B)
- new net: R2.1, SW1.3 (C)
- new net: R5.2, SW2.2 (B)
- new net: R11.2, U3.6 (CFG)
- new net: R4.1, SW2.3 (C)
- new net +3V3: C1.1, C3.1, R1.1, R2.2, R4.2, R7.1, R8.1, U1.3 (3V3), U4.4 (VREF)
- new net +9V: C10.2, C4.1, C9.1, D1.1 (K), J2.A4 (VBUS), J2.A9 (VBUS), J2.B4 (VBUS), J2.B9 (VBUS), R10.1, R9.1, U2.8 (VIN), U4.5 (VM)
- new net CC1: J2.A5 (CC1), R14.1, U3.4 (CC1)
- new net CC2: J2.B5 (CC2), R13.1, U3.5 (CC2)
- new net CLOSE_SW: SW2.1 (A), U1.5 (IO2)
- new net EN: C2.1, R1.2, U1.8 (EN)
- new net GND: C1.2, C10.1, C2.2, C3.2, C4.2, C5.2, C6.1, C7.2, C8.2, C9.2, J2.A1 (GND), J2.A12 (GND), J2.B1 (GND), J2.B12 (GND), J2.S1 (SHIELD), R12.2, R13.2, R14.2, R3.1, R5.1, R6.1, SW3.1, U1.1 (GND), U1.11 (GND), U1.14 (GND), U1.2 (GND), U1.36 (GND), U1.37 (GND), U1.38 (GND), U1.39 (GND), U1.40 (GND), U1.41 (GND), U1.42 (GND), U1.43 (GND), U1.44 (GND), U1.45 (GND), U1.46 (GND), U1.47 (GND), U1.48 (GND), U1.49 (GND), U1.50 (GND), U1.51 (GND), U1.52 (GND), U1.53 (GND), U2.2 (GND), U2.3 (GND), U2.9 (GND), U3.2 (GND), U4.1 (GND), U4.9 (GND)
- new net IO0: C6.2, U1.12 (IO0), Y1.1
- new net IO1: C7.1, U1.13 (IO1), Y1.2
- new net IO4: U1.9 (IO4)
- new net IO5: U1.10 (IO5)
- new net IO8: R7.2, U1.22 (IO8)
- new net IO9/BOOT: C5.1, R8.2, SW3.2, U1.23 (IO9)
- new net JTAG_DM: J2.A7 (D-), J2.B7 (D-), U1.17 (IO12)
- new net JTAG_DP: J2.A6 (D+), J2.B6 (D+), U1.18 (IO13)
- new net LED_CTRL: R6.2, U2.4 (CTRL)
- new net LPI2C_SCL: U1.16 (IO7)
- new net LPI2C_SDA: U1.15 (IO6)
- new net MOTOR_IN1: U1.26 (IO20), U4.3 (IN1)
- new net MOTOR_IN2: U1.27 (IO21), U4.2 (IN2)
- new net OPEN_SW: SW1.1 (A), U1.6 (IO3)
- new net STATE_LED: U1.19 (IO14)
- new net UART_RXD: U1.30 (RXD0)
- new net UART_TXD: U1.31 (TXD0)
- no-connect marks 0 -> 9
Other:
- note added: "* CL=12.5pF"
- note added: "* Inductor can also be PSPNAQ6045-470M"

Commit message: rev1: sync change
Parts:
- removed D1: SS24FL, Diode_SMD:D_SOD-123F, symbol Device:D
- removed R5, R6: 22k, Resistor_SMD:R_0402_1005Metric, symbol Device:R
- removed R9: 0.15R/0.5w, Resistor_SMD:R_0805_2012Metric, symbol Device:R
- removed U2: AL8860MP, Package_SO:MSOP-8-1EP_3x3mm_P0.65mm_EP1.5x1.8mm, symbol Driver_LED:AL8860MP
- removed Y1: 32.768k, Crystal:Crystal_SMD_3215-2Pin_3.2x1.5mm, symbol Device:Crystal
- added J2: UART_PROG, Connector_PinHeader_1.27mm:PinHeader_1x06_P1.27mm_Vertical, symbol Connector:Conn_01x06_Pin
- added Q1: AO3400A, Package_TO_SOT_SMD:SOT-23, symbol Transistor_FET:AO3400A
- added U2: AP63203WU, Package_TO_SOT_SMD:TSOT-23-6, symbol Regulator_Switching:AP63203WU
- C4: footprint Capacitor_SMD:C_0402_1005Metric -> Capacitor_SMD:C_0603_1608Metric; LCSC C1525 -> (none)
- C6: value 20pF -> 100nF; LCSC C1554 -> (none)
- C7: value 20pF -> 22uF; footprint Capacitor_SMD:C_0402_1005Metric -> Capacitor_SMD:C_0603_1608Metric; LCSC C1554 -> (none)
- J1: value LED -> LED_OUT
- L1: value 47uH -> 3.9uH; footprint Inductor_SMD:L_APV_ANR6045 -> Inductor_SMD:L_Changjiang_FNR3015S
- R8: renamed from R11; value 20k -> 47k
- renumbered J2 to J3, J3 to J4, R12 to R10, R14 to R11, R8 to R5, R7 to R6, R10 to R7, R13 to R9
Connections:
- net +9V is gone; now on net +12V: C10.2, C4.1, C9.1, J3.A4 (VBUS), J3.A9 (VBUS), J3.B4 (VBUS), J3.B9 (VBUS), R7.1, U4.5 (VM)
- net STATE_LED is gone; now on net LED_CTRL: U1.19 (IO14)
- net +3V3: now also C7.1, L1.2, SW1.3 (C), SW2.3 (C), J2.1 (Pin_1), U2.1 (FB); no longer R2.2, R4.2
- net CLOSE_SW: now also R3.2; no longer SW2.1 (A)
- net EN: now also J2.4 (Pin_4)
- net GND: now also R4.1, SW1.2 (B), SW2.2 (B), J2.6 (Pin_6), Q1.2 (S), U2.4 (GND); no longer C6.1, R3.1
- net IO9/BOOT: now also J2.5 (Pin_5)
- net LED_CTRL: now also R4.2, Q1.1 (G)
- net OPEN_SW: now also R2.2; no longer SW1.1 (A)
- net UART_RXD: now also J2.3 (Pin_3)
- net UART_TXD: now also J2.2 (Pin_2)
- net at L1.1: now also C6.2, U2.5 (SW); no longer J1.1 (Pin_1)
- net +12V: now reaches J1.2 (Pin_2)
- net +12V: now also U2.2 (EN), U2.3 (IN)
- net at R2.1: now also SW1.1 (A); no longer SW1.3 (C)
- net IO0: no longer names the net of U1.12 (IO0)
- net IO0: no longer C6.2
- net IO1: no longer names the net of U1.13 (IO1)
- net IO1: no longer C7.1
- net IO4: no longer names the net of U1.9 (IO4)
- net IO5: no longer names the net of U1.10 (IO5)
- net LPI2C_SCL: no longer names the net of U1.16 (IO7)
- net LPI2C_SDA: no longer names the net of U1.15 (IO6)
- new net: C6.1, U2.6 (BST)
- new net: J1.1 (Pin_1), Q1.3 (D)
- new net: R3.1, SW2.1 (A)
- no-connect marks 9 -> 15
Other:
- note removed: "* CL=12.5pF"
- note removed: "* Inductor can also be PSPNAQ6045-470M"
- moved on the sheet: C10, C5, C9, J4, R10, R5, SW3, U4
