File: flipcab-rounded.kicad_pcb (KiCad board)
At the start: 4 copper layers, 50 x 23 mm, 34 parts, among them J1 LED_OUT, J2 UART_PROG, J3 USB_JTAG, J4 MOTOR_OUT, Q1 AO3400A, SW1 OPEN_DET, SW2 CLOSE_DET, SW3 BOOT, U1 ESP32-C6-MINI-1, U2 AP63203WU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

Commit message: rev1: send off to JLC
Routing:
- net +12V: track 77.2 -> 78.9 mm
- net CC2: track 17.0 -> 16.3 mm
